Commit message: feat: add rviz display launch

File: urdf/abb_irb4600_40_255.xacro (robot description, xacro)
@@ -2,4 +2,5 @@
 <robot name="abb_irb4600_40_255" xmlns:xacro="http://wiki.ros.org/xacro">
   <xacro:include filename="$(find abb_irb4600_description)/urdf/abb_irb4600_40_255_macro.xacro"/>
+  <link name="world"/>
   <xacro:abb_irb4600_40_255 prefix=""/>
 </robot>
