Commit message: fix: correct joint naming convention in xacro file

File: urdf/abb_irb4600_40_255_macro.xacro (robot description, xacro)
@@ -156,5 +156,5 @@
       <origin xyz="0 0 0" rpy="0 0 0"/>
     </joint>
-    <joint name="${prefix}joint_1" type="revolute">
+    <joint name="joint_${prefix}1" type="revolute">
       <parent link="${prefix}base_link"/>
       <child link="${prefix}link_1"/>
@@ -164,5 +164,5 @@
       <dynamics damping="5.0" friction="0.2" />
     </joint>
-    <joint name="${prefix}joint_2" type="revolute">
+    <joint name="joint_${prefix}2" type="revolute">
       <parent link="${prefix}link_1"/>
       <child link="${prefix}link_2"/>
@@ -172,5 +172,5 @@
       <dynamics damping="5.0" friction="0.2" />
     </joint>
-    <joint name="${prefix}joint_3" type="revolute">
+    <joint name="joint_${prefix}3" type="revolute">
       <parent link="${prefix}link_2"/>
       <child link="${prefix}link_3"/>
@@ -180,5 +180,5 @@
       <dynamics damping="5.0" friction="0.2" />
     </joint>
-    <joint name="${prefix}joint_4" type="revolute">
+    <joint name="joint_${prefix}4" type="revolute">
       <parent link="${prefix}link_3"/>
       <child link="${prefix}link_4"/>
@@ -188,5 +188,5 @@
       <dynamics damping="5.0" friction="0.2" />
     </joint>
-    <joint name="${prefix}joint_5" type="revolute">
+    <joint name="joint_${prefix}5" type="revolute">
       <parent link="${prefix}link_4"/>
       <child link="${prefix}link_5"/>
@@ -196,5 +196,5 @@
       <dynamics damping="5.0" friction="0.2" />
     </joint>
-    <joint name="${prefix}joint_6" type="revolute">
+    <joint name="joint_${prefix}6" type="revolute">
       <parent link="${prefix}link_5"/>
       <child link="${prefix}link_6"/>

Commit message: compas_fab and visualization related updates

File: urdf/abb_irb4600_40_255_macro.xacro (robot description, xacro)
@@ -185,5 +185,5 @@
       <origin xyz="0.331 0 0.175" rpy="0 0 0"/>
       <axis xyz="1 0 0"/>
-      <limit lower="${radians(-400)}" upper="${radians(400)}" effort="10000" velocity="${radians(250)}" />
+      <limit lower="${radians(-200)}" upper="${radians(200)}" effort="10000" velocity="${radians(250)}" />
       <dynamics damping="5.0" friction="0.2" />
     </joint>
@@ -201,5 +201,5 @@
       <origin xyz="0.135 0 0" rpy="0 ${pi/2} 0"/>
       <axis xyz="0 0 1"/>
-      <limit lower="${radians(-400)}" upper="${radians(400)}" effort="100000" velocity="${radians(360)}" />
+      <limit lower="${radians(-200)}" upper="${radians(200)}" effort="100000" velocity="${radians(360)}" />
       <dynamics damping="5.0" friction="0.2" />
     </joint>
